Commit message: Add pybullet value plots

File: configs/pybullet/envs/assets/franka_panda/franka_panda_robotiq.urdf (robot description, URDF)
Before this commit: robot franka_panda, 21 links, 20 joints
Links:
- link left_inner_finger_pad_collision: geometry collision box size=0.022 0.00635 0.0575; visual box size=0.002 0.00035 0.0075
- link right_inner_finger_pad_collision: geometry collision box size=0.022 0.00635 0.0575; visual box size=0.002 0.00035 0.0075
